File: hardware/CDCEmu.brd (EAGLE design)
At the start: 61 x 41.9 mm, 99 parts, among them Q1 NPN, Q10 NCH, Q11 NPN, Q2 PCH, Q3 NPN, Q4 NPN, Q5 NPN, Q6 NPN, Q7 NCH, Q8 NCH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

Commit message: [HW] Correct resistor values
Parts:
- R1: value 1.5k -> 100k
- R10: value 1.5k -> 15k
- R11: value 200k -> 100k
- R12: value 68.1k -> 100k
- R15, R17, R19, R21, R31, R33: value 10k -> 100k
- R2: value 1.5k -> 10k
- R4: value 10k -> 240
- R5: value 10k -> 470
- R7: value 4.7k -> 47k
- R9: value 24.9k -> 100k
